Commit message: Sensors were added to robot

File: src/my_robot/urdf/project_robot.xacro (robot description, xacro)
@@ -55,3 +55,127 @@
     </visual>
   </link>
+<?Left wheel?>
+  <link name="left_wheel">
+        <visual name="left_wheel_visual">
+		<origin xyz="0 0 0" rpy=" 0 1.5707 1.5707"/>
+      		<geometry>
+        		<cylinder radius="0.1" length="0.05"/>
+      		</geometry>
+	</visual>
+	<collision name="left_wheel_collision">
+		<origin xyz="0 0 0" rpy=" 0 1.5707 1.5707"/>
+      		<geometry>
+        		<cylinder radius="0.1" length="0.05"/>
+      		</geometry>
+	</collision>
+	<inertial>
+      		<mass value="5.0"/>
+      		<origin xyz="0.0 0 0" rpy=" 0 0 0"/>
+      		<inertia
+          		ixx="0.1" ixy="0" ixz="0"
+          		iyy="0.1" iyz="0"
+          		izz="0.1" />
+    </inertial>
+  </link>
+<?Right wheel?>
+  <link name="right_wheel">
+        <visual name="right_wheel_visual">
+		<origin xyz="0 0 0" rpy=" 0 1.5707 1.5707"/>
+      		<geometry>
+        		<cylinder radius="0.1" length="0.05"/>
+      		</geometry>
+	</visual>
+	<collision name="right_wheel_collision">
+		<origin xyz="0 0 0" rpy=" 0 1.5707 1.5707"/>
+      		<geometry>
+        		<cylinder radius="0.1" length="0.05"/>
+      		</geometry>
+	</collision>
+	<inertial>
+      		<mass value="5.0"/>
+      		<origin xyz="0.0 0 0" rpy=" 0 0 0"/>
+      		<inertia
+          		ixx="0.1" ixy="0" ixz="0"
+          		iyy="0.1" iyz="0"
+          		izz="0.1" />
+    </inertial>
+  </link>
+<?Camera?>
+  <link name="camera">
+        <visual name="camera_visual">
+		<origin xyz="0 0 0" rpy=" 0 0 0"/>
+      		<geometry>
+        		<box size="0.05 0.05 0.05" />
+      		</geometry>
+	</visual>
+	<collision name="camera_collision">
+		<origin xyz="0 0 0" rpy=" 0 0 0"/>
+      		<geometry>
+        		<box size=".05 .05 .05"/>
+      		</geometry>
+	</collision>
+	<inertial>
+      		<mass value="0.1"/>
+      		<origin xyz="0 0 0" rpy=" 0 0 0"/>
+      		<inertia
+          		ixx="1e-6" ixy="0" ixz="0"
+          		iyy="1e-6" iyz="0"
+          		izz="1e-6" />
+    </inertial>
+  </link>
+<?Lidar?>
+  <link name="hokuyo">
+        <visual name="hokuyo_visual">
+		<origin xyz="0 0 0" rpy=" 0 0 0"/>
+      		<geometry>
+        		<mesh filename="package://my_robot/meshes/hokuyo.dae" />
+      		</geometry>
+	</visual>
+	<collision name="hokuyo_collision">
+		<origin xyz="0 0 0" rpy=" 0 0 0"/>
+      		<geometry>
+        		<box size=".1 .1 .1" filename="package://my_robot/meshes/hokuyo.dae" />
+      		</geometry>
+	</collision>
+	<inertial>
+      		<mass value="1e-5"/>
+      		<origin xyz="0 0 0" rpy=" 0 0 0"/>
+      		<inertia
+          		ixx="1e-6" ixy="0" ixz="0"
+          		iyy="1e-6" iyz="0"
+          		izz="1e-6" />
+    </inertial>
+  </link>
+<?left wheel joint?>
+  <joint type="continuous" name="left_wheel_hinge">
+	<origin xyz="0 0.15 0" rpy="0 0 0"/>
+    	<child link="left_wheel"/>
+    	<parent link="chassis"/>
+    	<axis xyz="0 1 0" rpy="0 0 0"/>
+    	<limit effort="10000" velocity="1000"/>
+    	<dynamics damping="1.0" friction="1.0"/>
+  </joint>
+<?right wheel joint?>
+  <joint type="continuous" name="right_wheel_hinge">
+	<origin xyz="0 -0.15 0" rpy="0 0 0"/>
+    	<child link="right_wheel"/>
+    	<parent link="chassis"/>
+    	<axis xyz="0 1 0" rpy="0 0 0"/>
+    	<limit effort="10000" velocity="1000"/>
+    	<dynamics damping="1.0" friction="1.0"/>
+  </joint>
+<?camera joint?>
+  <joint type="fixed" name="camera_joint">
+	<origin xyz="0.2 0 0" rpy="0 0 0"/>
+    	<child link="camera"/>
+    	<parent link="chassis"/>
+    	<axis xyz="0 1 0" rpy="0 0 0"/>
+  </joint>
+<?lidar joint?>
+  <joint type="fixed" name="hokuyo_joint">
+	<origin xyz="0.15 0 0.1" rpy="0 0 0"/>
+    	<child link="hokuyo"/>
+    	<parent link="chassis"/>
+    	<axis xyz="0 1 0" rpy="0 0 0"/>
+  </joint>
 </robot>
